File: Bai_channels.kicad_sch (KiCad schematic)
At the start: 120 parts, among them Q1 BC337, Q10 BC337, Q11 BC337, Q12 BC337, Q2 BC337, Q3 BC337, Q4 BC337, Q5 BC337, Q6 BC337, Q7 BC337, Q8 BC337, Q9 BC337, U1 ATmega328-P, U3 LM7805_TO220

Commit message: changes
Parts:
- removed U15, U21, U27, U9: ~, symbol Custom_Symbol_Lib:VB
- added D32: LED, symbol Device:LED
- added R33: R, symbol Device:R
Connections:
- net at Q5.1 (C), R11.2, R16.2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: now also R33.2
- net at D31.2 (A), Q7.3 (E), U33.1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: now also D32.2 (A)
- net at 16MHz1.2, C2.1, U1.10 (XTAL2/PB7): no longer 16MHz1.1, C3.1, U1.9 (XTAL1/PB6)
- new net: D32.1 (K), R33.1
- new net: 16MHz1.1, C3.1, U1.9 (XTAL1/PB6)

Commit message: vibration motor footprint
Parts:
- added C1: 10µF, Custom_FP_Lib:Through-Hole Cap, symbol Device:C_Polarized
- RV1: footprint (none) -> Potentiometer_THT:Potentiometer_Alps_RK163_Single_Horizontal
Connections:
- net at C1.1, R4.2, RV1.3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: now also 16MHz1.2, C2.1, U1.10 (XTAL2/PB7), C1.1
- net at C1.2, C1.2, C2.2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: now also C1.2
Changed lines of the file:
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@@
   (junction (at 208.28 90.17) (diameter 0) (color 0 0 0 0)
   )
+  (junction (at 49.53 86.36) (diameter 0) (color 0 0 0 0)
+  )
   (junction (at 200.66 110.49) (diameter 0) (color 0 0 0 0)
   )
@@
   (junction (at 182.88 76.2) (diameter 0) (color 0 0 0 0)
   )
+  (junction (at 93.98 129.54) (diameter 0) (color 0 0 0 0)
+  )
   (junction (at 246.38 62.23) (diameter 0) (color 0 0 0 0)
   )
@@
   (junction (at 182.88 86.36) (diameter 0) (color 0 0 0 0)
   )
+  (junction (at 49.53 163.83) (diameter 0) (color 0 0 0 0)
+  )
   (junction (at 233.68 86.36) (diameter 0) (color 0 0 0 0)
   )
@@
     (stroke (width 0) (type default))
   )
+  (wire (pts (xy 49.53 86.36) (xy 66.04 86.36))
+    (stroke (width 0) (type default))
+  )
   (wire (pts (xy 246.38 100.33) (xy 246.38 104.14))
     (stroke (width 0) (type default))
@@
     (stroke (width 0) (type default))
   )
+  (wire (pts (xy 93.98 129.54) (xy 93.98 156.21))
+    (stroke (width 0) (type default))
+  )
   (wire (pts (xy 213.36 82.55) (xy 215.9 82.55))
     (stroke (width 0) (type default))
@@
     (stroke (width 0) (type default))
   )
-  (wire (pts (xy 45.72 163.83) (xy 66.04 163.83))
+  (wire (pts (xy 45.72 163.83) (xy 49.53 163.83))
     (stroke (width 0) (type default))
   )
@@
     (stroke (width 0) (type default))
   )
+  (wire (pts (xy 49.53 125.73) (xy 49.53 163.83))
+    (stroke (width 0) (type default))
+  )
   (wire (pts (xy 81.28 158.75) (xy 238.76 158.75))
     (stroke (width 0) (type default))
@@
     (stroke (width 0) (type default))
   )
-  (wire (pts (xy 45.72 86.36) (xy 66.04 86.36))
+  (wire (pts (xy 45.72 86.36) (xy 49.53 86.36))
     (stroke (width 0) (type default))
   )
@@
     (stroke (width 0) (type default))
   )
+  (wire (pts (xy 49.53 163.83) (xy 66.04 163.83))
+    (stroke (width 0) (type default))
+  )
   (wire (pts (xy 182.88 163.83) (xy 104.14 163.83))
     (stroke (width 0) (type default))
@@
     (stroke (width 0) (type default))
   )
+  (wire (pts (xy 49.53 86.36) (xy 49.53 118.11))
+    (stroke (width 0) (type default))
+  )
   (wire (pts (xy 29.21 128.27) (xy 29.21 163.83))
     (stroke (width 0) (type default))
@@
     (stroke (width 0) (type default))
   )
-  (wire (pts (xy 93.98 86.36) (xy 93.98 156.21))
+  (wire (pts (xy 93.98 86.36) (xy 93.98 129.54))
     (stroke (width 0) (type default))
   )
@@
       (effects (font (size 1.27 1.27)) (justify right))
     )
-    (property "Footprint" "" (at 104.14 90.17 0)
+    (property "Footprint" "Potentiometer_THT:Potentiometer_Alps_RK163_Single_Horizontal" (at 104.14 90.17 0)
       (effects (font (size 1.27 1.27)) hide)
     )
@@
         )
       )
+    )
+  )
+  (symbol (lib_id "Device:C_Polarized") (at 49.53 121.92 0) (unit 1)
+    (in_bom yes) (on_board yes) (dnp no) (fields_autoplaced)
+    (property "Reference" "C1" (at 53.34 119.761 0)
+      (effects (font (size 1.27 1.27)) (justify left))
+    )
+    (property "Value" "10µF" (at 53.34 122.301 0)
+      (effects (font (size 1.27 1.27)) (justify left))
+    )
+    (property "Footprint" "Custom_FP_Lib:Through-Hole Cap" (at 50.4952 125.73 0)
+      (effects (font (size 1.27 1.27)) hide)
+    )
+    (property "Datasheet" "~" (at 49.53 121.92 0)
+      (effects (font (size 1.27 1.27)) hide)
+    )
+    (pin "1")
+    (pin "2")
+    (instances
+      (project "Test_1_V1"
+        (path "/8943c65c-643a-4659-9240-617acc1f3f5e"
+          (reference "C1") (unit 1)
+        )
+      )
+      (project "Bai_channels"
+        (path "/9a6b30ab-2d97-4b8c-9c1f-d1e56c330002"
+          (reference "C5") (unit 1)
+        )
+      )

Commit message: save
Parts:
- U10, U11, U12, U13, U14, U16, U17, U18, U19, U20, U22, U23, U24, U25, U26, U28, U29, U30, U31, U32, U33, U34, U35, U36, U37, U38, U39, U4, U5, U6, U7, U8: footprint (none) -> custom:vibration_motor
Changed lines of the file:
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@@
       (effects (font (size 1.27 1.27)))
     )
-    (property "Footprint" "" (at 203.2 114.3 0)
+    (property "Footprint" "custom:vibration_motor" (at 203.2 114.3 0)
       (effects (font (size 1.27 1.27)) hide)
     )
@@
       (effects (font (size 1.27 1.27)))
     )
-    (property "Footprint" "" (at 228.6 72.39 0)
+    (property "Footprint" "custom:vibration_motor" (at 228.6 72.39 0)
       (effects (font (size 1.27 1.27)) hide)
     )
@@
       (effects (font (size 1.27 1.27)))
     )
-    (property "Footprint" "" (at 241.3 72.39 0)
+    (property "Footprint" "custom:vibration_motor" (at 241.3 72.39 0)
       (effects (font (size 1.27 1.27)) hide)
     )
@@
       (effects (font (size 1.27 1.27)))
     )
-    (property "Footprint" "" (at 177.8 58.42 0)
+    (property "Footprint" "custom:vibration_motor" (at 177.8 58.42 0)
       (effects (font (size 1.27 1.27)) hide)
     )
@@
       (effects (font (size 1.27 1.27)))
     )
-    (property "Footprint" "" (at 228.6 128.27 0)
+    (property "Footprint" "custom:vibration_motor" (at 228.6 128.27 0)
       (effects (font (size 1.27 1.27)) hide)
     )
@@
       (effects (font (size 1.27 1.27)))
     )
-    (property "Footprint" "" (at 177.8 114.3 0)
+    (property "Footprint" "custom:vibration_motor" (at 177.8 114.3 0)
       (effects (font (size 1.27 1.27)) hide)
     )
@@
       (effects (font (size 1.27 1.27)))
     )
-    (property "Footprint" "" (at 190.5 72.39 0)
+    (property "Footprint" "custom:vibration_motor" (at 190.5 72.39 0)
       (effects (font (size 1.27 1.27)) hide)
     )
@@
       (effects (font (size 1.27 1.27)))
     )
-    (property "Footprint" "" (at 228.6 100.33 0)
+    (property "Footprint" "custom:vibration_motor" (at 228.6 100.33 0)
       (effects (font (size 1.27 1.27)) hide)
     )
@@
       (effects (font (size 1.27 1.27)))
     )
-    (property "Footprint" "" (at 215.9 114.3 0)
+    (property "Footprint" "custom:vibration_motor" (at 215.9 114.3 0)
       (effects (font (size 1.27 1.27)) hide)
     )
@@
       (effects (font (size 1.27 1.27)))
     )
-    (property "Footprint" "" (at 228.6 86.36 0)
+    (property "Footprint" "custom:vibration_motor" (at 228.6 86.36 0)
       (effects (font (size 1.27 1.27)) hide)
     )
@@
       (effects (font (size 1.27 1.27)))
     )
-    (property "Footprint" "" (at 203.2 72.39 0)
+    (property "Footprint" "custom:vibration_motor" (at 203.2 72.39 0)
       (effects (font (size 1.27 1.27)) hide)
     )
@@
       (effects (font (size 1.27 1.27)))
     )
-    (property "Footprint" "" (at 203.2 86.36 0)
+    (property "Footprint" "custom:vibration_motor" (at 203.2 86.36 0)
       (effects (font (size 1.27 1.27)) hide)
     )
@@
       (effects (font (size 1.27 1.27)))
     )
-    (property "Footprint" "" (at 215.9 72.39 0)
+    (property "Footprint" "custom:vibration_motor" (at 215.9 72.39 0)
       (effects (font (size 1.27 1.27)) hide)
     )
@@
       (effects (font (size 1.27 1.27)))
     )
-    (property "Footprint" "" (at 241.3 114.3 0)
+    (property "Footprint" "custom:vibration_motor" (at 241.3 114.3 0)
       (effects (font (size 1.27 1.27)) hide)
     )
@@
       (effects (font (size 1.27 1.27)))
     )
-    (property "Footprint" "" (at 177.8 100.33 0)
+    (property "Footprint" "custom:vibration_motor" (at 177.8 100.33 0)
       (effects (font (size 1.27 1.27)) hide)
     )
@@
       (effects (font (size 1.27 1.27)))
     )
-    (property "Footprint" "" (at 215.9 58.42 0)
+    (property "Footprint" "custom:vibration_motor" (at 215.9 58.42 0)
       (effects (font (size 1.27 1.27)) hide)
     )
@@
       (effects (font (size 1.27 1.27)))
     )
-    (property "Footprint" "" (at 177.8 72.39 0)
+    (property "Footprint" "custom:vibration_motor" (at 177.8 72.39 0)
       (effects (font (size 1.27 1.27)) hide)
     )
@@
       (effects (font (size 1.27 1.27)))
     )
-    (property "Footprint" "" (at 190.5 58.42 0)
+    (property "Footprint" "custom:vibration_motor" (at 190.5 58.42 0)
       (effects (font (size 1.27 1.27)) hide)
     )
@@
       (effects (font (size 1.27 1.27)))
     )
-    (property "Footprint" "" (at 215.9 100.33 0)
+    (property "Footprint" "custom:vibration_motor" (at 215.9 100.33 0)
       (effects (font (size 1.27 1.27)) hide)
     )
@@
       (effects (font (size 1.27 1.27)))
     )
-    (property "Footprint" "" (at 190.5 100.33 0)
+    (property "Footprint" "custom:vibration_motor" (at 190.5 100.33 0)
       (effects (font (size 1.27 1.27)) hide)
     )
@@
       (effects (font (size 1.27 1.27)))
     )
-    (property "Footprint" "" (at 241.3 86.36 0)
+    (property "Footprint" "custom:vibration_motor" (at 241.3 86.36 0)
       (effects (font (size 1.27 1.27)) hide)
     )
@@
       (effects (font (size 1.27 1.27)))
     )
-    (property "Footprint" "" (at 190.5 86.36 0)
+    (property "Footprint" "custom:vibration_motor" (at 190.5 86.36 0)
       (effects (font (size 1.27 1.27)) hide)
     )
@@
       (effects (font (size 1.27 1.27)))
     )
-    (property "Footprint" "" (at 241.3 58.42 0)
+    (property "Footprint" "custom:vibration_motor" (at 241.3 58.42 0)
       (effects (font (size 1.27 1.27)) hide)
     )
@@
       (effects (font (size 1.27 1.27)))
     )
-    (property "Footprint" "" (at 228.6 58.42 0)
+    (property "Footprint" "custom:vibration_motor" (at 228.6 58.42 0)
       (effects (font (size 1.27 1.27)) hide)
     )
@@
       (effects (font (size 1.27 1.27)))
     )
-    (property "Footprint" "" (at 215.9 86.36 0)
+    (property "Footprint" "custom:vibration_motor" (at 215.9 86.36 0)
       (effects (font (size 1.27 1.27)) hide)
     )
@@
       (effects (font (size 1.27 1.27)))
     )
-    (property "Footprint" "" (at 241.3 128.27 0)
+    (property "Footprint" "custom:vibration_motor" (at 241.3 128.27 0)
       (effects (font (size 1.27 1.27)) hide)
     )
@@
       (effects (font (size 1.27 1.27)))
     )
-    (property "Footprint" "" (at 203.2 100.33 0)
+    (property "Footprint" "custom:vibration_motor" (at 203.2 100.33 0)
       (effects (font (size 1.27 1.27)) hide)
     )
@@
       (effects (font (size 1.27 1.27)))
     )
-    (property "Footprint" "" (at 190.5 114.3 0)
+    (property "Footprint" "custom:vibration_motor" (at 190.5 114.3 0)
       (effects (font (size 1.27 1.27)) hide)
     )
@@
       (effects (font (size 1.27 1.27)))
     )
-    (property "Footprint" "" (at 241.3 100.33 0)
+    (property "Footprint" "custom:vibration_motor" (at 241.3 100.33 0)
       (effects (font (size 1.27 1.27)) hide)
     )
@@
       (effects (font (size 1.27 1.27)))
     )
-    (property "Footprint" "" (at 177.8 86.36 0)
+    (property "Footprint" "custom:vibration_motor" (at 177.8 86.36 0)
       (effects (font (size 1.27 1.27)) hide)
     )
@@
       (effects (font (size 1.27 1.27)))
     )
-    (property "Footprint" "" (at 228.6 114.3 0)
+    (property "Footprint" "custom:vibration_motor" (at 228.6 114.3 0)
       (effects (font (size 1.27 1.27)) hide)
     )
@@
       (effects (font (size 1.27 1.27)))
     )
-    (property "Footprint" "" (at 203.2 58.42 0)
-      (effects (font (size 1.27 1.27)) hide)
-    )
+    (property "Footprint" "custom:vibration_motor" (at 203.2 58.42 0)
+      (effects (font (size 1.27 1.27)) hide)
+    )

Commit message: led footprints
Parts:
- D1, D10, D11, D12, D13, D14, D15, D16, D17, D18, D19, D2, D20, D21, D22, D23, D24, D25, D26, D27, D28, D29, D3, D30, D31, D32, D4, D5, D6, D7, D8, D9: footprint (none) -> custom:LED
Changed lines of the file:
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@@
       (effects (font (size 1.27 1.27)) (justify right) hide)
     )
-    (property "Footprint" "" (at 175.26 114.3 0)
+    (property "Footprint" "custom:LED" (at 175.26 114.3 0)
       (effects (font (size 1.27 1.27)) hide)
     )
@@
       (effects (font (size 1.27 1.27)) (justify right) hide)
     )
-    (property "Footprint" "" (at 175.26 86.36 0)
+    (property "Footprint" "custom:LED" (at 175.26 86.36 0)
       (effects (font (size 1.27 1.27)) hide)
     )
@@
       (effects (font (size 1.27 1.27)) (justify right) hide)
     )
-    (property "Footprint" "" (at 175.26 100.33 0)
+    (property "Footprint" "custom:LED" (at 175.26 100.33 0)
       (effects (font (size 1.27 1.27)) hide)
     )
@@
       (effects (font (size 1.27 1.27)) (justify right) hide)
     )
-    (property "Footprint" "" (at 226.06 100.33 0)
+    (property "Footprint" "custom:LED" (at 226.06 100.33 0)
       (effects (font (size 1.27 1.27)) hide)
     )
@@
       (effects (font (size 1.27 1.27)) (justify right) hide)
     )
-    (property "Footprint" "" (at 226.06 114.3 0)
+    (property "Footprint" "custom:LED" (at 226.06 114.3 0)
       (effects (font (size 1.27 1.27)) hide)
     )
@@
       (effects (font (size 1.27 1.27)) (justify right) hide)
     )
-    (property "Footprint" "" (at 238.76 114.3 0)
+    (property "Footprint" "custom:LED" (at 238.76 114.3 0)
       (effects (font (size 1.27 1.27)) hide)
     )
@@
       (effects (font (size 1.27 1.27)) (justify right) hide)
     )
-    (property "Footprint" "" (at 200.66 114.3 0)
+    (property "Footprint" "custom:LED" (at 200.66 114.3 0)
       (effects (font (size 1.27 1.27)) hide)
     )
@@
       (effects (font (size 1.27 1.27)) (justify right) hide)
     )
-    (property "Footprint" "" (at 226.06 86.36 0)
+    (property "Footprint" "custom:LED" (at 226.06 86.36 0)
       (effects (font (size 1.27 1.27)) hide)
     )
@@
       (effects (font (size 1.27 1.27)) (justify right) hide)
     )
-    (property "Footprint" "" (at 238.76 58.42 0)
+    (property "Footprint" "custom:LED" (at 238.76 58.42 0)
       (effects (font (size 1.27 1.27)) hide)
     )
@@
       (effects (font (size 1.27 1.27)) (justify right) hide)
     )
-    (property "Footprint" "" (at 200.66 58.42 0)
+    (property "Footprint" "custom:LED" (at 200.66 58.42 0)
       (effects (font (size 1.27 1.27)) hide)
     )
@@
       (effects (font (size 1.27 1.27)) (justify right) hide)
     )
-    (property "Footprint" "" (at 238.76 72.39 0)
+    (property "Footprint" "custom:LED" (at 238.76 72.39 0)
       (effects (font (size 1.27 1.27)) hide)
     )
@@
       (effects (font (size 1.27 1.27)) (justify right) hide)
     )
-    (property "Footprint" "" (at 200.66 86.36 0)
+    (property "Footprint" "custom:LED" (at 200.66 86.36 0)
       (effects (font (size 1.27 1.27)) hide)
     )
@@
       (effects (font (size 1.27 1.27)) (justify right) hide)
     )
-    (property "Footprint" "" (at 213.36 114.3 0)
+    (property "Footprint" "custom:LED" (at 213.36 114.3 0)
       (effects (font (size 1.27 1.27)) hide)
     )
@@
       (effects (font (size 1.27 1.27)) (justify right) hide)
     )
-    (property "Footprint" "" (at 175.26 72.39 0)
+    (property "Footprint" "custom:LED" (at 175.26 72.39 0)
       (effects (font (size 1.27 1.27)) hide)
     )
@@
       (effects (font (size 1.27 1.27)) (justify right) hide)
     )
-    (property "Footprint" "" (at 200.66 72.39 0)
+    (property "Footprint" "custom:LED" (at 200.66 72.39 0)
       (effects (font (size 1.27 1.27)) hide)
     )
@@
       (effects (font (size 1.27 1.27)) (justify right) hide)
     )
-    (property "Footprint" "" (at 213.36 86.36 0)
+    (property "Footprint" "custom:LED" (at 213.36 86.36 0)
       (effects (font (size 1.27 1.27)) hide)
     )
@@
       (effects (font (size 1.27 1.27)) (justify right) hide)
     )
-    (property "Footprint" "" (at 213.36 58.42 0)
+    (property "Footprint" "custom:LED" (at 213.36 58.42 0)
       (effects (font (size 1.27 1.27)) hide)
     )
@@
       (effects (font (size 1.27 1.27)) (justify right) hide)
     )
-    (property "Footprint" "" (at 187.96 100.33 0)
+    (property "Footprint" "custom:LED" (at 187.96 100.33 0)
       (effects (font (size 1.27 1.27)) hide)
     )
@@
       (effects (font (size 1.27 1.27)) (justify right) hide)
     )
-    (property "Footprint" "" (at 187.96 86.36 0)
+    (property "Footprint" "custom:LED" (at 187.96 86.36 0)
       (effects (font (size 1.27 1.27)) hide)
     )
@@
       (effects (font (size 1.27 1.27)) (justify right) hide)
     )
-    (property "Footprint" "" (at 213.36 100.33 0)
+    (property "Footprint" "custom:LED" (at 213.36 100.33 0)
       (effects (font (size 1.27 1.27)) hide)
     )
@@
       (effects (font (size 1.27 1.27)) (justify right) hide)
     )
-    (property "Footprint" "" (at 226.06 58.42 0)
+    (property "Footprint" "custom:LED" (at 226.06 58.42 0)
       (effects (font (size 1.27 1.27)) hide)
     )
@@
       (effects (font (size 1.27 1.27)) (justify right) hide)
     )
-    (property "Footprint" "" (at 226.06 72.39 0)
+    (property "Footprint" "custom:LED" (at 226.06 72.39 0)
       (effects (font (size 1.27 1.27)) hide)
     )
@@
       (effects (font (size 1.27 1.27)) (justify right) hide)
     )
-    (property "Footprint" "" (at 200.66 100.33 0)
+    (property "Footprint" "custom:LED" (at 200.66 100.33 0)
       (effects (font (size 1.27 1.27)) hide)
     )
@@
       (effects (font (size 1.27 1.27)) (justify right) hide)
     )
-    (property "Footprint" "" (at 238.76 128.27 0)
+    (property "Footprint" "custom:LED" (at 238.76 128.27 0)
       (effects (font (size 1.27 1.27)) hide)
     )
@@
       (effects (font (size 1.27 1.27)) (justify right) hide)
     )
-    (property "Footprint" "" (at 187.96 58.42 0)
+    (property "Footprint" "custom:LED" (at 187.96 58.42 0)
       (effects (font (size 1.27 1.27)) hide)
     )
@@
       (effects (font (size 1.27 1.27)) (justify right) hide)
     )
-    (property "Footprint" "" (at 238.76 86.36 0)
+    (property "Footprint" "custom:LED" (at 238.76 86.36 0)
       (effects (font (size 1.27 1.27)) hide)
     )
@@
       (effects (font (size 1.27 1.27)) (justify right) hide)
     )
-    (property "Footprint" "" (at 187.96 72.39 0)
+    (property "Footprint" "custom:LED" (at 187.96 72.39 0)
       (effects (font (size 1.27 1.27)) hide)
     )
@@
       (effects (font (size 1.27 1.27)) (justify right) hide)
     )
-    (property "Footprint" "" (at 213.36 72.39 0)
+    (property "Footprint" "custom:LED" (at 213.36 72.39 0)
       (effects (font (size 1.27 1.27)) hide)
     )
@@
       (effects (font (size 1.27 1.27)) (justify right) hide)
     )
-    (property "Footprint" "" (at 238.76 100.33 0)
+    (property "Footprint" "custom:LED" (at 238.76 100.33 0)
       (effects (font (size 1.27 1.27)) hide)
     )
@@
       (effects (font (size 1.27 1.27)) (justify right) hide)
     )
-    (property "Footprint" "" (at 172.72 58.42 0)
+    (property "Footprint" "custom:LED" (at 172.72 58.42 0)
       (effects (font (size 1.27 1.27)) hide)
     )
@@
       (effects (font (size 1.27 1.27)) (justify right) hide)
     )
-    (property "Footprint" "" (at 187.96 114.3 0)
+    (property "Footprint" "custom:LED" (at 187.96 114.3 0)
       (effects (font (size 1.27 1.27)) hide)
     )
@@
       (effects (font (size 1.27 1.27)) (justify right) hide)
     )
-    (property "Footprint" "" (at 226.06 128.27 0)
-      (effects (font (size 1.27 1.27)) hide)
-    )
+    (property "Footprint" "custom:LED" (at 226.06 128.27 0)
+      (effects (font (size 1.27 1.27)) hide)
+    )
