File: Bai_channels.kicad_sch (KiCad schematic)
At the start: 24 parts, among them J2 5019514000, U1 ATmega328-P, U2 LM7805_TO220

Commit message: 16 channel
Parts:
- removed 16MHz1: Crystal, Crystal:Crystal_HC49-4H_Vertical, symbol Device:Crystal
- removed C1: 10µF, custom:capacitor, symbol Device:C_Polarized
- removed C2, C3: 22pF, custom:capacitor, symbol Device:C
- removed R4: 10kR, custom:R, symbol Device:R
- removed U1: ATmega328-P, Package_DIP:DIP-28_W7.62mm_Socket, symbol MCU_Microchip_ATmega:ATmega328-P
Connections:
- net at C1.2, C1.2, C1.2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: now also J2.17; no longer J2.33
- net at U1.11 (PD5): no longer J2.25
- net at U1.12 (PD6): no longer J2.26
- net at U1.17 (PB3): no longer J2.17
- net at U1.18 (PB4): no longer J2.18
- net at U1.19 (PB5): no longer J2.19
- net at U1.2 (PD0): no longer J2.20
- net at U1.3 (PD1): no longer J2.21
- net at U1.4 (PD2): no longer J2.22
- net at U1.5 (PD3): no longer J2.23
- net at U1.6 (PD4): no longer J2.24

Commit message: work
Connections:
- net at C1.2, C1.2, C1.2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: now also J2.32; no longer J2.17
Changed lines of the file:
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@@
-    (stroke (width 0) (type default))
-  )
-  (wire (pts (xy 231.14 67.31) (xy 271.78 67.31))
     (stroke (width 0) (type default))
   )
@@
     (stroke (width 0) (type default))
   )
+  (wire (pts (xy 105.41 95.25) (xy 264.16 95.25))
+    (stroke (width 0) (type default))
+  )
   (wire (pts (xy 110.49 64.77) (xy 222.25 64.77))
     (stroke (width 0) (type default))
@@
     (stroke (width 0) (type default))
   )
+  (wire (pts (xy 264.16 95.25) (xy 264.16 105.41))
+    (stroke (width 0) (type default))
+  )
   (wire (pts (xy 91.44 60.96) (xy 96.52 60.96))
     (stroke (width 0) (type default))
@@
     (stroke (width 0) (type default))
   )
-  (wire (pts (xy 105.41 95.25) (xy 231.14 95.25))
-    (stroke (width 0) (type default))
-  )
   (wire (pts (xy 82.55 26.67) (xy 271.78 26.67))
     (stroke (width 0) (type default))
@@
     (stroke (width 0) (type default))
   )
+  (wire (pts (xy 264.16 105.41) (xy 271.78 105.41))
+    (stroke (width 0) (type default))
+  )
   (wire (pts (xy 227.33 69.85) (xy 227.33 59.69))
     (stroke (width 0) (type default))
@@
     (stroke (width 0) (type default))
   )
-  (wire (pts (xy 231.14 95.25) (xy 231.14 67.31))
-    (stroke (width 0) (type default))
-  )

Commit message: final track
Connections:
- net at J2.11: no longer U1.6 (PD4)
- net at J2.27: now also U1.6 (PD4)
Changed lines of the file:
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@@
+    (stroke (width 0) (type default))
+  )
+  (wire (pts (xy 266.7 92.71) (xy 271.78 92.71))
     (stroke (width 0) (type default))
   )
@@
     (stroke (width 0) (type default))
   )
+  (wire (pts (xy 266.7 52.07) (xy 266.7 92.71))
+    (stroke (width 0) (type default))
+  )
   (wire (pts (xy 107.95 72.39) (xy 107.95 62.23))
     (stroke (width 0) (type default))
@@
     (stroke (width 0) (type default))
   )
+  (wire (pts (xy 223.52 52.07) (xy 266.7 52.07))
+    (stroke (width 0) (type default))
+  )
   (wire (pts (xy 46.99 17.78) (xy 50.8 17.78))
     (stroke (width 0) (type default))
@@
     (stroke (width 0) (type default))
   )
-  (wire (pts (xy 223.52 52.07) (xy 271.78 52.07))
-    (stroke (width 0) (type default))
-  )

Commit message: final design
Parts:
- removed J2: 5019514000, custom:CON_5019514000, symbol Custom_Symbol_Lib:5019514000
- added J1: 5020782510, CON_5020782510, symbol 2024-03-11_19-24-41:5020782510
- added J2: Conn_01x02_Pin, custom:pinHeader, symbol Connector:Conn_01x02_Pin
Connections:
- net at C1.2, C1.2, C1.2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: now also J1.19, J1.23, J1.6
- net at U1.14 (PB0): now also J1.14
- net at U1.15 (PB1): now also J1.18
- net at U1.16 (PB2): now also J1.20
- net at U1.14 (PB0): now also J1.1
- net at U1.5 (PD3): now also J1.10
- net at U1.11 (PD5): now also J1.12
- net at U1.12 (PD6): now also J1.16
- net at U1.15 (PB1): now also J1.2
- net at U1.6 (PD4): now also J1.25
- net at U1.16 (PB2): now also J1.3
- net at U1.17 (PB3): now also J1.4
- net at U1.18 (PB4): now also J1.5
- net at U1.19 (PB5): now also J1.24
- net at U1.2 (PD0): now also J1.7
- net at U1.3 (PD1): now also J1.8
- net at U1.4 (PD2): now also J1.22
- new net: J1.17, J2.1 (Pin_1)
- new net: J1.21, J2.2 (Pin_2)
