File: Bai_channels.kicad_pcb (KiCad board)
At the start: 2 copper layers, 18 parts, among them J2 5019514000, U2 LM7805_TO220, U3 ATmega328-P, U4 ATmega328-P

Commit message: final track
Connections:
- J2 pad 11: Net-(U3-PD4) -> unconnected-(J2-Pad11)
- J2 pad 27: unconnected-(J2-Pad27) -> Net-(U3-PD4)
Routing:
- net Net-(U1-VCC): track 0.00 -> 92.9 mm, vias 0 -> 1
- net Net-(U1-GND): track 48.4 -> 134.6 mm, vias 0 -> 2
- net Net-(U2-VO): track 30.6 -> 97.3 mm, vias 1 -> 2
- net Net-(U4-XTAL2/PB7): track 0.00 -> 35.1 mm, vias 0 -> 1
- net Net-(U4-XTAL1/PB6): track 0.00 -> 19.1 mm
- net Net-(U3-PD7): track 0.00 -> 18.3 mm
- net Net-(U4-~{RESET}/PC6): track 0.00 -> 12.4 mm
- net Net-(U3-PC0): track 0.00 -> 11.0 mm
- net Net-(U3-PD4): track 0.00 -> 2.88 mm

Commit message: design complete
Parts:
- moved J2 30.1 mm to (158.4, 96.6)
- moved C3 30.1 mm to (137.7, 86.3)
- moved U1 30.1 mm to (141.7, 81.6)
- moved U3 30.1 mm to (154.4, 113.4)
- moved 16MHz1 30.1 mm to (142.0, 86.9)
- moved 16MHz2 30.1 mm to (176.3, 96.0)
- moved C1 30.1 mm to (177.3, 79.1)
- moved C2 30.1 mm to (135.1, 84.1)
- moved C4 30.1 mm to (177.3, 86.7)
- moved C5 30.1 mm to (135.1, 95.6)
- moved C6 30.1 mm to (135.1, 88.4)
- moved C7 30.1 mm to (177.3, 81.6)
- moved C8 30.1 mm to (177.3, 91.5)
- moved R1 30.1 mm to (137.6, 88.7)
- moved R2 30.1 mm to (174.8, 84.1)
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Routing:
- net Net-(U3-PC0): track 11.0 -> 92.0 mm, vias 0 -> 2
Other:
- board outline added: 45.9 x 38.2 mm

Commit message: final design
Parts:
- added J1: 5020782510, Library:CON_5020782510, F.Cu at (159.2, 97.6)
- J2: value 5019514000 -> Conn_01x02_Pin; footprint custom:CON_5019514000 -> custom:pinHeader
- moved J2 15.3 mm to (160.0, 111.8), turned to 0 degrees
Connections:
- J2 pad 1: Net-(U3-PB0) -> Net-(J2-Pin_1)
- J2 pad 2: Net-(U3-PB1) -> Net-(J2-Pin_2)
Routing:
- net Net-(U3-PD1): track 61.3 -> 16.2 mm, vias 3 -> 1
- net Net-(U3-PD3): track 44.4 -> 9.65 mm, vias 2 -> 1
- net Net-(J2-Pin_1): track 0.00 -> 30.3 mm, vias 0 -> 2
- net Net-(J2-Pin_2): track 0.00 -> 25.2 mm, vias 0 -> 2
- net Net-(U3-PC0): track 92.0 -> 67.1 mm, vias 2 -> 0
- net Net-(U4-PB1): track 46.8 -> 25.4 mm
- net Net-(U1-GND): track 134.6 -> 120.9 mm, vias 2 -> 3
- net Net-(U3-PB5): track 36.6 -> 24.8 mm, vias 2 -> 3
- net Net-(U3-PD6): track 11.0 -> 20.9 mm
- net Net-(U3-PD2): track 20.2 -> 12.1 mm, vias 1 -> 0
- net Net-(U1-VCC): track 92.9 -> 85.9 mm, vias 1 -> 0
- net Net-(U3-PB2): track 14.1 -> 20.1 mm, vias 1 -> 0
- net Net-(U3-PD5): track 13.6 -> 19.6 mm, vias 1 -> 2
- net Net-(U3-PB3): track 26.7 -> 21.5 mm, vias 0 -> 1
- net Net-(U4-PB2): track 29.6 -> 24.4 mm, vias 1 -> 5
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